File: ANDON_Terminal_DL_v2/ANDON_v2.kicad_pcb (KiCad board)
At the start: 2 copper layers, 69.1 x 126.1 mm, 41 parts, among them P15 CONN_5X2, P4 CONN_5, P5 CONN_8, P8 CONN_4, Q1 TIP127, Q2 TIP127, Q3 TIP127, Q4 TIP127, SW1 SW_PUSH, U1 ULN2003A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

Commit message: PIC PROGRAMMING CONNECTOR MODIFICATION
Parts:
- removed the ? at (126.8, 151.4)
- added P2: PRG_CONN, SIL-5, F.Cu at (126.6, 151.2)
Routing:
- net /PGC: track 62.4 -> 49.3 mm
- net /PGD: track 57.1 -> 52.0 mm
- net /RESET: track 42.1 -> 43.1 mm
